Commit message: F

File: jackal_description/urdf/jackal.urdf.xacro (robot description, xacro)
@@ -236,3 +236,28 @@
   <!-- Optional for Clearpath internal softwares -->
   <xacro:include filename="$(optenv CPR_URDF_EXTRAS empty.urdf)" />
+  <xacro:arg name="gpu" default="false"/>
+  <xacro:property name="gpu" value="$(arg gpu)" />
+  <xacro:arg name="organize_cloud" default="false"/>
+  <xacro:property name="organize_cloud" value="$(arg organize_cloud)" />
+  <xacro:include filename="$(find velodyne_description)/urdf/VLP-16.urdf.xacro"/>
+  <xacro:VLP-16 parent="base_link" name="velodyne" topic="/velodyne_points" hz="10" samples="440" gpu="${gpu}">
+    <origin xyz="0.12 0 0.26" rpy="0 0 0" />
+  </xacro:VLP-16>
+  <!-- Velodyne mount stuff -->
+  <link name="velodyne_mount">
+    <visual>
+      <origin xyz="0.001 0.001 0.07" rpy="0.0 0.0 -1.57" />
+      <geometry>
+        <mesh filename="package://jackal_description/meshes/vlp_mount_final.stl" scale="0.001 0.001 0.001"/>
+      </geometry>
+      <material name="aluminum" >
+        <color rgba="0.45 0.45 0.45 1"/>
+      </material>
+    </visual>
+  </link>
+  <joint name="velodyne_mount_joint" type="fixed">
+    <parent link="front_mount" />
+    <child link="velodyne_mount" />
+    <origin xyz="0 0 0.0" />
+  </joint>
 </robot>
